File: teensy3.6-cs42448.sch (EAGLE design)
At the start: 17 parts, among them U1 CS42448

Commit message: Add files via upload
Connections:
- net GND: now also U1.AD0/!CS!
- net LEFT: now also C3.1
- net N$1: now also R2.1
- net N$10: now also R3.2, R4.1
- net N$11: now also C2.-, R4.2
- net N$7: now also C1.-, R2.2
- net RIGHT: now also C2.+, C4.1

Commit message: Add files via upload
Parts:
- added C10, C9: 100nf, Seeed-Capacitor:CERAMIC-100NF-50V-10%-X7R(0805)
- added C11, C14: 10nf, Seeed-Capacitor:CERAMIC-10NF-50V-5%-X7R(0805)
- added C8: 10uf, Seeed-Capacitor:CERAMIC-10UF-25V-10%-X5R(0805)
- added R1, R5: 2K, OPL_Resistor:SMD-RES-2K-5%-1/10W(0603)
- added SJ1, SJ2: (no value), jumper:SJ
- added U$2: CAT811T, CAT811T:CAT811T
Connections:
- new net 3.3V: R1.2, U$2.VCC
- new net N$25: R5.2, SJ2.2
- new net N$26: U$2.RESET, U1.!RST!
- net 3V3: no longer U1.!RST!
- net AGND: now also R1.1; no longer U1.AOUT1-, U1.AOUT2-, U1.AOUT3-, U1.AOUT4-, U1.AOUT5-, U1.AOUT6-, U1.AOUT7-, U1.AOUT8-
- net GND: now also C10.1, C11.1, C14.1, C8.1, C9.1, R5.1, U$2.GND; no longer U1.AD0/!CS!, U1.AUX_SCLK
- net N$1: now also R1.2
- net N$10: now also U1.AIN6+/AIN6A; no longer U1.AIN5-/AIN5B
- net N$11: now also SJ1.2, SJ2.1, U1.AD0/!CS!; no longer U1.AIN6+/AIN6A
- net N$12: now also R1.1, SJ1.1; no longer U1.AIN6-/AIN6B
- net N$17: now also R1.2
- net N$6: now also C10.2, C11.2, C14.2, C8.2, C9.2
Other:
- moved on the sheet: FB1, R3
